File: hardware/barnabas_noggin_V4.sch (EAGLE design)
At the start: 59 parts, among them J1 POWER_JACKPTH, J10 2.54mm, J2 ICSP, J3 ICSP, J4 USB-mini-90 -SMD, J5 ICSP, J6 2.54mm, J7 2.54mm, J8 2.54mm, J9 2.54mm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

Commit message: Modify silkscreen text. Update logo pattern.
Parts:
- J1: PARTNO (none) -> EJ508A
- J10, J8: PARTNO (none) -> PPTC081LFBN-RC
- J2, J3, J5: PARTNO (none) -> M20-9980346
- J4: PARTNO (none) -> UJ2-MBH-1-SMT-TR
- J6, J7, J9: PARTNO (none) -> M20-7820646
- PB1, PB2: PARTNO (none) -> PTS820 J15M SMTR LFS
- U3: PARTNO (none) -> LP2985-33DBVR
Changed lines of the file:
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@@
 <part name="U$13" library="barnabas_noggin_V4" deviceset="GND" device=""/>
 <part name="U$16" library="barnabas_noggin_V4" deviceset="GND" device=""/>
-<part name="PB1" library="barnabas_noggin_V4" deviceset="PUSHBUTTON" device="" value="157SW"/>
+<part name="PB1" library="barnabas_noggin_V4" deviceset="PUSHBUTTON" device="" value="157SW">
+<attribute name="PARTNO" value="PTS820 J15M SMTR LFS"/>
+</part>
 <part name="U$28" library="barnabas_noggin_V4" deviceset="GND" device=""/>
 <part name="U$31" library="barnabas_noggin_V4" deviceset="5V" device=""/>
@@
 </part>
 <part name="U$3" library="barnabas_noggin_V4" deviceset="GND" device=""/>
-<part name="J4" library="barnabas_noggin_V4" deviceset="CONNECTOR_USB_MINI-B" device="" value="USB-mini-90 -SMD"/>
+<part name="J4" library="barnabas_noggin_V4" deviceset="CONNECTOR_USB_MINI-B" device="" value="USB-mini-90 -SMD">
+<attribute name="PARTNO" value="UJ2-MBH-1-SMT-TR"/>
+</part>
 <part name="U$6" library="barnabas_noggin_V4" deviceset="GND" device=""/>
 <part name="U$7" library="barnabas_noggin_V4" deviceset="GND" device=""/>
@@
 <part name="U$5" library="barnabas_noggin_V4" deviceset="GND" device=""/>
 <part name="U$12" library="barnabas_noggin_V4" deviceset="5V_PIN" device=""/>
-<part name="J5" library="barnabas_noggin_V4" deviceset="CONNECTOR_2X3" device="" value="ICSP"/>
+<part name="J5" library="barnabas_noggin_V4" deviceset="CONNECTOR_2X3" device="" value="ICSP">
+<attribute name="PARTNO" value="M20-9980346"/>
+</part>
 <part name="R1" library="barnabas_noggin_V4" deviceset="RESISTOR" device="0603" value="1K">
 <attribute name="PARTNO" value="RC0603FR-071KL "/>
@@
 </part>
 <part name="U$8" library="barnabas_noggin_V4" deviceset="5V_PIN" device=""/>
-<part name="J1" library="barnabas_noggin_V4" deviceset="POWER_JACK" device="PTH"/>
+<part name="J1" library="barnabas_noggin_V4" deviceset="POWER_JACK" device="PTH">
+<attribute name="PARTNO" value="EJ508A"/>
+</part>
 <part name="D1" library="barnabas_noggin_V4" deviceset="SCHOTTKY_DIODE" device="" value="SS1P3L">
 <attribute name="PARTNO" value="SS1P3L-M3/84A"/>
@@
 <part name="R3" library="barnabas_noggin_V4" deviceset="RESISTOR" device="" value="470"/>
 <part name="E2" library="barnabas_noggin_V4" deviceset="BUZZER" device=""/>
-<part name="J2" library="barnabas_noggin_V4" deviceset="CONNECTOR_2X3" device="" value="ICSP"/>
-<part name="J3" library="barnabas_noggin_V4" deviceset="CONNECTOR_2X3" device="" value="ICSP"/>
-<part name="J8" library="barnabas_noggin_V4" deviceset="PINHD-1X8" device="" value="2.54mm"/>
-<part name="J10" library="barnabas_noggin_V4" deviceset="PINHD-1X8" device="" value="2.54mm"/>
-<part name="J7" library="barnabas_noggin_V4" deviceset="PINHD-1X6" device="" value="2.54mm"/>
-<part name="J9" library="barnabas_noggin_V4" deviceset="PINHD-1X6" device="" value="2.54mm"/>
+<part name="J2" library="barnabas_noggin_V4" deviceset="CONNECTOR_2X3" device="" value="ICSP">
+<attribute name="PARTNO" value="M20-9980346"/>
+</part>
+<part name="J3" library="barnabas_noggin_V4" deviceset="CONNECTOR_2X3" device="" value="ICSP">
+<attribute name="PARTNO" value="M20-9980346"/>
+</part>
+<part name="J8" library="barnabas_noggin_V4" deviceset="PINHD-1X8" device="" value="2.54mm">
+<attribute name="PARTNO" value="PPTC081LFBN-RC"/>
+</part>
+<part name="J10" library="barnabas_noggin_V4" deviceset="PINHD-1X8" device="" value="2.54mm">
+<attribute name="PARTNO" value="PPTC081LFBN-RC"/>
+</part>
+<part name="J7" library="barnabas_noggin_V4" deviceset="PINHD-1X6" device="" value="2.54mm">
+<attribute name="PARTNO" value="M20-7820646"/>
+</part>
+<part name="J9" library="barnabas_noggin_V4" deviceset="PINHD-1X6" device="" value="2.54mm">
+<attribute name="PARTNO" value="M20-7820646"/>
+</part>
 <part name="C7" library="barnabas_noggin_V4" deviceset="CAPACITOR_100NF_0603" device="" value="100nF">
 <attribute name="PARTNO" value="CC0603ZRY5V9BB104"/>
@@
 <attribute name="PARTNO" value="MF-FSMF050X-2"/>
 </part>
-<part name="PB2" library="barnabas_noggin_V4" deviceset="PUSHBUTTON" device="" value="157SW"/>
+<part name="PB2" library="barnabas_noggin_V4" deviceset="PUSHBUTTON" device="" value="157SW">
+<attribute name="PARTNO" value="PTS820 J15M SMTR LFS"/>
+</part>
 <part name="U$40" library="barnabas_noggin_V4" deviceset="GND" device=""/>
-<part name="J6" library="barnabas_noggin_V4" deviceset="PINHD-1X6" device="" value="2.54mm"/>
+<part name="J6" library="barnabas_noggin_V4" deviceset="PINHD-1X6" device="" value="2.54mm">
+<attribute name="PARTNO" value="M20-7820646"/>
+</part>
 <part name="U5" library="barnabas_noggin_V4" deviceset="L9110S_DRIVER" device=""/>
 <part name="U$1" library="barnabas_noggin_V4" deviceset="5V_PIN" device=""/>
@@
 <part name="U$42" library="barnabas_noggin_V4" deviceset="5V" device=""/>
 <part name="U$43" library="barnabas_noggin_V4" deviceset="5V" device=""/>
-<part name="U3" library="barnabas_noggin_V4" deviceset="LP2985-XXDBVR" device=""/>
+<part name="U3" library="barnabas_noggin_V4" deviceset="LP2985-XXDBVR" device="">
+<attribute name="PARTNO" value="LP2985-33DBVR"/>
+</part>
 <part name="U$44" library="barnabas_noggin_V4" deviceset="GND" device=""/>
 <part name="U$45" library="barnabas_noggin_V4" deviceset="GND" device=""/>
@@
 <instance part="U$13" gate="G$1" x="33.02" y="154.94"/>
 <instance part="U$16" gate="G$1" x="35.56" y="111.76"/>
-<instance part="PB1" gate="G$1" x="27.94" y="170.18"/>
+<instance part="PB1" gate="G$1" x="27.94" y="170.18">
+<attribute name="PARTNO" x="27.94" y="170.18" size="1.778" layer="96" display="off"/>
+</instance>
 <instance part="U$28" gate="G$1" x="10.16" y="165.1"/>
 <instance part="U$31" gate="G$1" x="48.26" y="190.5"/>
@@
 </instance>
 <instance part="U$3" gate="G$1" x="218.44" y="114.3"/>
-<instance part="J4" gate="G$1" x="198.374" y="139.7" rot="MR0"/>
+<instance part="J4" gate="G$1" x="198.374" y="139.7" rot="MR0">
+<attribute name="PARTNO" x="198.374" y="139.7" size="1.778" layer="96" rot="MR0" display="off"/>
+</instance>
 <instance part="U$6" gate="G$1" x="211.074" y="114.3"/>
 <instance part="U$7" gate="G$1" x="182.88" y="114.3"/>
@@
 <instance part="U$5" gate="G$1" x="222.25" y="16.51"/>
 <instance part="U$12" gate="G$1" x="222.25" y="36.83"/>
-<instance part="J5" gate="A" x="209.55" y="26.67"/>
+<instance part="J5" gate="A" x="209.55" y="26.67">
+<attribute name="PARTNO" x="209.55" y="26.67" size="1.778" layer="96" display="off"/>
+</instance>
 <instance part="R1" gate="G$1" x="48.26" y="180.34" rot="R90">
 <attribute name="PARTNO" x="48.26" y="180.34" size="1.778" layer="96" rot="R90" display="off"/>
@@
 </instance>
 <instance part="U$8" gate="G$1" x="100.584" y="85.09"/>
-<instance part="J1" gate="G$1" x="17.78" y="27.94"/>
+<instance part="J1" gate="G$1" x="17.78" y="27.94">
+<attribute name="PARTNO" x="17.78" y="27.94" size="1.778" layer="96" display="off"/>
+</instance>
 <instance part="D1" gate="G$1" x="28.956" y="35.56">
 <attribute name="PARTNO" x="28.956" y="35.56" size="1.778" layer="96" display="off"/>
@@
 <instance part="R3" gate="G$1" x="81.28" y="17.78"/>
 <instance part="E2" gate="1" x="93.98" y="20.32"/>
-<instance part="J2" gate="A" x="144.78" y="30.48"/>
-<instance part="J3" gate="A" x="144.78" y="15.24"/>
-<instance part="J8" gate="A" x="317.5" y="154.94"/>
-<instance part="J10" gate="A" x="335.28" y="154.94"/>
-<instance part="J7" gate="A" x="314.96" y="127"/>
-<instance part="J9" gate="A" x="328.93" y="127.254"/>
+<instance part="J2" gate="A" x="144.78" y="30.48">
+<attribute name="PARTNO" x="144.78" y="30.48" size="1.778" layer="96" display="off"/>
+</instance>
+<instance part="J3" gate="A" x="144.78" y="15.24">
+<attribute name="PARTNO" x="144.78" y="15.24" size="1.778" layer="96" display="off"/>
+</instance>
+<instance part="J8" gate="A" x="317.5" y="154.94">
+<attribute name="PARTNO" x="317.5" y="154.94" size="1.778" layer="96" display="off"/>
+</instance>
+<instance part="J10" gate="A" x="335.28" y="154.94">
+<attribute name="PARTNO" x="335.28" y="154.94" size="1.778" layer="96" display="off"/>
+</instance>
+<instance part="J7" gate="A" x="314.96" y="127">
+<attribute name="PARTNO" x="314.96" y="127" size="1.778" layer="96" display="off"/>
+</instance>
+<instance part="J9" gate="A" x="328.93" y="127.254">
+<attribute name="PARTNO" x="328.93" y="127.254" size="1.778" layer="96" display="off"/>
+</instance>
 <instance part="C7" gate="G$1" x="134.62" y="76.2">
 <attribute name="PARTNO" x="134.62" y="76.2" size="1.778" layer="96" display="off"/>
@@
 <attribute name="PARTNO" x="100.584" y="73.66" size="1.778" layer="96" display="off"/>
 </instance>
-<instance part="PB2" gate="G$1" x="134.112" y="121.92"/>
+<instance part="PB2" gate="G$1" x="134.112" y="121.92">
+<attribute name="PARTNO" x="134.112" y="121.92" size="1.778" layer="96" display="off"/>
+</instance>
 <instance part="U$40" gate="G$1" x="147.32" y="114.3"/>
-<instance part="J6" gate="A" x="284.48" y="72.39"/>
+<instance part="J6" gate="A" x="284.48" y="72.39">
+<attribute name="PARTNO" x="284.48" y="72.39" size="1.778" layer="96" display="off"/>
+</instance>
 <instance part="U5" gate="G$1" x="294.64" y="63.5"/>
 <instance part="U$1" gate="G$1" x="264.16" y="86.36"/>
@@
 <instance part="U$42" gate="G$1" x="90.17" y="85.09"/>
 <instance part="U$43" gate="G$1" x="187.96" y="86.36"/>
-<instance part="U3" gate="G$1" x="205.74" y="76.2"/>
+<instance part="U3" gate="G$1" x="205.74" y="76.2">
+<attribute name="PARTNO" x="205.74" y="76.2" size="1.778" layer="96" display="off"/>
+</instance>
 <instance part="U$44" gate="G$1" x="187.96" y="63.5"/>
 <instance part="U$45" gate="G$1" x="226.06" y="63.5"/>
